Commit message: add gripper aligned frame to urdf

File: models/iiwa/iiwa_description/iiwa14_schunk_gripper.urdf (robot description, URDF)
Before this commit: robot iiwa14, 14 links, 13 joints
Links:
- added link iiwa_link_ee_gripper_aligned
Joints:
- added joint tool1_joint: type fixed, parent iiwa_link_ee, child iiwa_link_ee_gripper_aligned, origin xyz=0 0 0.0 rpy=0.0  0.39259999999999995 1.5699999999999998

Commit message: Remove our schunk models and point to Drake's instead

File: models/iiwa/iiwa_description/iiwa14_schunk_gripper.urdf (robot description, URDF)
Before this commit: robot iiwa14, 15 links, 14 joints
Links:
- removed link palm
- removed link wsg_50_finger_left_link
- removed link wsg_50_finger_right_link
- added link wsg_50_base_link, mass 1.2; collision mesh filename=package://wsg_50_description/meshes/WSG50_110.obj scale=1 1 1; visual mesh filename=package://wsg_50_description/meshes/WSG50_110.obj scale=1 1 1
- added link wsg_50_finger_left, mass 0.1; collision mesh filename=package://wsg_50_description/meshes/WSG-FMF.obj scale=0.001 0.001 0.001; visual mesh filename=package://wsg_50_description/meshes/WSG-FMF.obj scale=0.001 0.001 0.001
- added link wsg_50_finger_right, mass 0.1; collision mesh filename=package://wsg_50_description/meshes/WSG-FMF.obj scale=0.001 0.001 0.001; visual mesh filename=package://wsg_50_description/meshes/WSG-FMF.obj scale=0.001 0.001 0.001
- added link wsg_50_gripper_left, mass 0.1; collision mesh filename=package://wsg_50_description/meshes/GUIDE_WSG50_110.obj scale=0.001 0.001 0.001; visual mesh filename=package://wsg_50_description/meshes/GUIDE_WSG50_110.obj scale=0.001 0.001 0.001
- added link wsg_50_gripper_right, mass 0.1; collision mesh filename=package://wsg_50_description/meshes/GUIDE_WSG50_110.obj scale=0.001 0.001 0.001; visual mesh filename=package://wsg_50_description/meshes/GUIDE_WSG50_110.obj scale=0.001 0.001 0.001
Joints:
- removed joint gripper_mount_joint
- removed joint wsg_50_finger_left_joint
- removed joint wsg_50_finger_right_joint
- added joint wsg_50_base_joint_gripper_left: type prismatic, parent wsg_50_base_link, child wsg_50_gripper_left, origin xyz=0 0 0 rpy=0 0 0, axis 1 0 0, limit lower=-0.055 upper=-0.0027 effort=1.0 velocity=1.0
- added joint wsg_50_base_joint_gripper_right: type prismatic, parent wsg_50_base_link, child wsg_50_gripper_right, origin xyz=0 0 0 rpy=0 0 3.14159, axis -1 0 0, limit lower=0.0027 upper=0.055 effort=1.0 velocity=1.0
- added joint wsg_50_guide_joint_finger_left: type fixed, parent wsg_50_gripper_left, child wsg_50_finger_left, origin xyz=0 0 0.023 rpy=0 0 0, axis 1 0 0, limit effort=100 velocity=100
- added joint wsg_50_guide_joint_finger_right: type fixed, parent wsg_50_gripper_right, child wsg_50_finger_right, origin xyz=0 0 0.023 rpy=0 0 0, axis 1 0 0, limit effort=100 velocity=100
- added joint wsg_50_mount_joint: type fixed, parent iiwa_link_ee, child wsg_50_base_link, origin xyz=0.005 0 0 rpy=1.57079632679 0 1.57079632679, axis 0 0 1

File: models/iiwa/iiwa_description/iiwa14_schunk_gripper_drake_sim.urdf (robot description, URDF)
Before this commit: robot iiwa14, 14 links, 13 joints
Links:
- removed link palm
- removed link wsg_50_finger_left_link
- removed link wsg_50_finger_right_link
- added link wsg_50_base_link, mass 1.2; collision mesh filename=package://wsg_50_description/meshes/WSG50_110.obj scale=1 1 1; visual mesh filename=package://wsg_50_description/meshes/WSG50_110.obj scale=1 1 1
- added link wsg_50_finger_left, mass 0.1; collision mesh filename=package://wsg_50_description/meshes/WSG-FMF.obj scale=0.001 0.001 0.001; visual mesh filename=package://wsg_50_description/meshes/WSG-FMF.obj scale=0.001 0.001 0.001
- added link wsg_50_finger_right, mass 0.1; collision mesh filename=package://wsg_50_description/meshes/WSG-FMF.obj scale=0.001 0.001 0.001; visual mesh filename=package://wsg_50_description/meshes/WSG-FMF.obj scale=0.001 0.001 0.001
- added link wsg_50_gripper_left, mass 0.1; collision mesh filename=package://wsg_50_description/meshes/GUIDE_WSG50_110.obj scale=0.001 0.001 0.001; visual mesh filename=package://wsg_50_description/meshes/GUIDE_WSG50_110.obj scale=0.001 0.001 0.001
- added link wsg_50_gripper_right, mass 0.1; collision mesh filename=package://wsg_50_description/meshes/GUIDE_WSG50_110.obj scale=0.001 0.001 0.001; visual mesh filename=package://wsg_50_description/meshes/GUIDE_WSG50_110.obj scale=0.001 0.001 0.001
Joints:
- removed joint gripper_mount_joint
- removed joint wsg_50_finger_left_joint
- removed joint wsg_50_finger_right_joint
- added joint wsg_50_base_joint_gripper_left: type prismatic, parent wsg_50_base_link, child wsg_50_gripper_left, origin xyz=0 0 0 rpy=0 0 0, axis 1 0 0, limit lower=-0.055 upper=-0.0027 effort=1.0 velocity=1.0
- added joint wsg_50_base_joint_gripper_right: type prismatic, parent wsg_50_base_link, child wsg_50_gripper_right, origin xyz=0 0 0 rpy=0 0 3.14159, axis -1 0 0, limit lower=0.0027 upper=0.055 effort=1.0 velocity=1.0
- added joint wsg_50_guide_joint_finger_left: type fixed, parent wsg_50_gripper_left, child wsg_50_finger_left, origin xyz=0 0 0.023 rpy=0 0 0, axis 1 0 0, limit effort=100 velocity=100
- added joint wsg_50_guide_joint_finger_right: type fixed, parent wsg_50_gripper_right, child wsg_50_finger_right, origin xyz=0 0 0.023 rpy=0 0 0, axis 1 0 0, limit effort=100 velocity=100
- added joint wsg_50_mount_joint: type fixed, parent iiwa_link_ee, child wsg_50_base_link, origin xyz=0.005 0 0 rpy=1.57079632679 0 1.57079632679, axis 0 0 1

Commit message: Add ghost palm frame for old calibs to work

File: models/iiwa/iiwa_description/iiwa14_schunk_gripper.urdf (robot description, URDF)
Before this commit: robot iiwa14, 17 links, 16 joints
Links:
- added link wsg_50_old_palm
Joints:
- added joint wsg_50_old_palm_joint: type fixed, parent iiwa_link_ee, child wsg_50_old_palm, origin xyz=0.02 0 0 rpy=0.0 0.3926 1.57079632679, axis 0 0 1
- joint wsg_50_mount_joint: origin xyz=0.005 0 0 rpy=1.57079632679 0 1.57079632679 -> xyz=0.005 0 0 rpy=1.57079632679 0.3926 1.57079632679

File: models/iiwa/iiwa_description/iiwa14_schunk_gripper_drake_sim.urdf (robot description, URDF)
Before this commit: robot iiwa14, 16 links, 15 joints
Links:
- added link wsg_50_old_palm
Joints:
- added joint wsg_50_old_palm_joint: type fixed, parent iiwa_link_ee, child wsg_50_old_palm, origin xyz=0.02 0 0 rpy=0.0 0.3926 1.57079632679, axis 0 0 1
- joint wsg_50_mount_joint: origin xyz=0.005 0 0 rpy=1.57079632679 0 1.57079632679 -> xyz=0.005 0 0 rpy=1.57079632679 0.3926 1.57079632679
