Commit message: working gelsight sim

File: models/iiwa/iiwa_description/iiwa14_schunk_gripper_with_gelsight.urdf (robot description, URDF)
Before this commit: robot iiwa14, 19 links, 18 joints
Joints:
- joint gelsight_joint: origin xyz=-0.012 0 0.112 rpy=0 1.57 0 -> xyz=-0.011 0 0.112 rpy=0 1.57 0
