Commit message: Tweaks to get rack simulation working

File: models/dishes/dish_rack_simple.urdf (robot description, URDF)
Before this commit: robot dish_rack_simple, 1 links, 0 joints
Links:
- link dish_rack_simple: mass 2 -> 0

Commit message: RGBD rendering, better collision on gripper

File: models/dishes/dish_rack_simple.urdf (robot description, URDF)
Before this commit: robot dish_rack_simple, 1 links, 0 joints
Links:
- link dish_rack_simple: mass 0 -> 5

File: models/rlg_misc_models/white_bin.urdf (robot description, URDF)
Before this commit: robot white_bin, 1 links, 0 joints
Links:
- link white_bin: mass 1 -> 2
